File: PCB/keyboard.kicad_sch (KiCad schematic)
At the start: 242 parts, among them J1 OLED_I2C_CON, SW1 SW_Push, SW10 SW_Push, SW100 SW_Push, SW101 SW_Push, SW102 SW_Push, SW103 SW_Push, SW104 SW_Push, SW107 SW_Push, SW108 SW_Push, SW109 SW_Push, SW11 SW_Push, SW110 SW_Push, SW111 SW_Push, SW112 SW_Push, SW114 RotaryEncoder_Switch, SW115 RotaryEncoder_Switch, SW12 SW_Push, SW13 SW_Push, SW14 SW_Push, SW15 SW_Push, SW16 SW_Push, SW17 SW_Push, SW18 SW_Push, SW19 SW_Push, SW2 SW_Push, SW20 SW_Push, SW21 SW_Push, SW22 SW_Push, SW23 SW_Push, SW24 SW_Push, SW25 SW_Push, SW26 SW_Push, SW27 SW_Push, SW28 SW_Push, SW29 SW_Push, SW3 SW_Push, SW30 SW_Push, SW31 SW_Push, SW32 SW_Push, SW33 SW_Push, SW34 SW_Push, SW35 SW_Push, SW36 SW_Push, SW37 SW_Push, SW38 SW_Push, SW39 SW_Push, SW4 SW_Push, SW40 SW_Push, SW41 SW_Push, SW42 SW_Push, SW43 SW_Push, SW44 SW_Push, SW45 SW_Push, SW46 SW_Push, SW47 SW_Push, SW48 SW_Push, SW49 SW_Push, SW5 SW_Push, SW50 SW_Push, SW51 SW_Push, SW52 SW_Push, SW53 SW_Push, SW54 SW_Push, SW55 SW_Push, SW56 SW_Push, SW57 SW_Push, SW58 SW_Push, SW59 SW_Push, SW6 SW_Push, SW60 SW_Push, SW61 SW_Push, SW62 SW_Push, SW63 SW_Push, SW64 SW_Push, SW65 SW_Push, SW66 SW_Push, SW67 SW_Push, SW68 SW_Push, SW69 SW_Push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

Commit message: First iteration
Parts:
- removed D104, D112, D32, D80, D88, D96: D, symbol Device:D
- removed SW104, SW112, SW32, SW80, SW88, SW96: SW_Push, symbol Switch:SW_Push
- C1, C2: footprint (none) -> Capacitor_THT:C_Disc_D5.0mm_W2.5mm_P5.00mm
- C3: footprint (none) -> Capacitor_THT:CP_Radial_D8.0mm_P3.50mm
- D1, D10, D100, D101, D102, D103, D105, D106, D107, D108, D109, D11, D110, D111, D12, D13, D14, D15, D16, D17, D18, D19, D2, D20, D21, D22, D23, D24, D25, D26, D27, D28, D29, D3, D30, D31, D33, D34, D35, D36, D37, D38, D39, D4, D40, D41, D42, D43, D44, D45, D46, D47, D48, D49, D5, D50, D51, D52, D53, D54, D55, D56, D57, D58, D59, D6, D60, D61, D62, D63, D64, D65, D66, D67, D68, D69, D7, D70, D71, D72, D73, D74, D75, D76, D77, D78, D79, D8, D81, D82, D83, D84, D85, D86, D87, D89, D9, D90, D91, D92, D93, D94, D95, D97, D98, D99: footprint (none) -> Diode_THT:D_DO-35_SOD27_P7.62mm_Horizontal
- SW1, SW10, SW100, SW101, SW102, SW103, SW107, SW108, SW109, SW11, SW110, SW111, SW12, SW13, SW14, SW15, SW16, SW17, SW18, SW19, SW2, SW20, SW21, SW22, SW23, SW24, SW25, SW26, SW27, SW28, SW29, SW3, SW30, SW31, SW33, SW34, SW35, SW36, SW37, SW38, SW39, SW4, SW40, SW41, SW42, SW43, SW44, SW45, SW46, SW47, SW48, SW49, SW5, SW50, SW51, SW52, SW53, SW54, SW55, SW56, SW57, SW58, SW59, SW6, SW60, SW61, SW62, SW63, SW64, SW65, SW66, SW67, SW68, SW69, SW7, SW70, SW71, SW72, SW73, SW74, SW75, SW76, SW77, SW78, SW79, SW8, SW81, SW82, SW83, SW84, SW85, SW86, SW87, SW89, SW9, SW90, SW91, SW92, SW93, SW94, SW95, SW97, SW98, SW99: footprint (none) -> Button_Switch_Keyboard:SW_Cherry_MX_1.00u_PCB
- SW114, SW115: footprint (none) -> Rotary_Encoder:RotaryEncoder_Alps_EC12E-Switch_Vertical_H20mm
- U4: footprint SN74AHCT125N:DIP794W45P254L1930H508Q14 -> KEYBOARD:DIP794W45P254L1930H508Q14
- U5: footprint (none) -> KEYBOARD:SOIC127P600X175-16N
- U6: value a -> 74HC595; footprint (none) -> KEYBOARD:SOIC127P600X175-16N
Connections:
- net GND: now also D114.3 (VDD), D115.3 (VDD), D116.3 (VDD)
- net RES1-A: now also A1.15 (GPIO11)
- net RES1-B: now also A1.16 (GPIO12)
- net RES2-A: now also A1.17 (GPIO13)
- net RES2-B: now also A1.19 (GPIO14)
- net RGB5: now also D122.2 (DIN); no longer D113.2 (DIN)
- net VBUS: now also D119.1 (VSS), D120.1 (VSS), D121.1 (VSS)
- net at D121.4 (DOUT): no longer D122.2 (DIN)
- net at D122.4 (DOUT): now also D113.2 (DIN)
- no-connect marks 0 -> 31
